Commit message: Oct17th C6rviz

File: c6/src/urdf1/urdf/urdf/demo1.urdf (robot description, URDF)
Before this commit: robot car, 2 links, 1 joints
Links:
- added link stick; visual cylinder length=0.5 radius=0.01
- link base_link: geometry visual box size=1 1 1
- link camera_link: geometry visual cylinder length=0.05 radius=0.2
Joints:
- removed joint base_link_to_map
- added joint camera_link_to_stick: type continuous, parent stick, child camera_link, origin xyz=0 0 0.275, axis 0 1 0, limit lower=-1.57 upper=1.57 effort=100 velocity=1
- added joint stick_to_base_link: type fixed, parent base_link, child stick, origin xyz=0 0 0.5 rpy=0 0 0
