Commit message: Oct19th gazebo&rviz-xacro

File: c6/xacrotest/src/xacrotest/urdf/all.urdf (robot description, URDF)
Before this commit: robot include_test, 9 links, 8 joints
Joints:
- joint camera2base_link: axis (none) -> 0 0 1; type fixed -> revolute

File: c6/xacrotest/src/xacrotest/xacro/camera.xacro (robot description, xacro)
@@ -18,8 +18,9 @@
         </visual>
     </link>
-    <joint name="camera2base_link" type="fixed">
+    <joint name="camera2base_link" type="revolute">
         <parent link="base_link" />
         <child link="camera" />
         <origin xyz="${camera_x} ${camera_y} ${camera_z}" />
+        <axis xyz="0 0 1" />
     </joint>
 </robot>
